File: SMT_ASSY/Lily58.sch (KiCad schematic (older format))
At the start: 83 parts, among them J1 LED, J2 4PIN, P1 i2c_pin, P2 i2c_pin, P3 ICSP, P4 OLED, SW1 SW_PUSH, SW10 SW_PUSH, SW11 SW_PUSH, SW12 SW_PUSH, SW13 SW_PUSH, SW14 SW_PUSH, SW15 SW_PUSH, SW16 SW_PUSH, SW17 SW_PUSH, SW18 SW_PUSH, SW19 SW_PUSH, SW2 SW_PUSH, SW20 SW_PUSH, SW21 SW_PUSH, SW22 SW_PUSH, SW23 SW_PUSH, SW24 SW_PUSH, SW25 SW_PUSH, SW26 SW_PUSH, SW27 SW_PUSH, SW28 SW_PUSH, SW29 SW_PUSH, SW3 SW_PUSH, SW4 SW_PUSH, SW5 SW_PUSH, SW6 SW_PUSH, SW7 SW_PUSH, SW8 SW_PUSH, SW9 SW_PUSH, U1 ProMicro

Commit message: Updated to use my lib (mostly)
Parts:
- removed J1: LED, Lily58-footprint:StripLED, symbol Lily58-rescue:LED-Lily58-cache
- added DISP0: OLED_128x32, Keyboard_Footprints:OLED, symbol Keyboard_Symbols:OLED_128x32
- added F0: PFC, Fuse:Fuse_1210_3225Metric, symbol Device:Polyfuse_Small
- added J0: USB_B_Micro, Connector_USB:USB_Micro-B_Molex-105017-0001, symbol Connector:USB_B_Micro
- added R0: 1.5k, Keyboard_Footprints:R_0603, symbol Device:R_Small_US
- added U0: USBLC6-2SC6, Package_TO_SOT_SMD:SOT-23-6, symbol Power_Protection:USBLC6-2SC6
- D1, D10, D11, D12, D13, D14, D15, D16, D17, D18, D19, D2, D20, D21, D22, D23, D24, D25, D26, D27, D28, D29, D3, D4, D5, D6, D7, D8, D9: footprint Lily58-footprint:Diode_TH_SOD123 -> Keyboard_Footprints:D_SOD-123_Flipped; symbol Lily58-rescue:D-Lily58-cache -> Keyboard_Symbols:Diode
- P3: symbol Lily58-rescue:CONN_01X06-Lily58-cache -> Connector_Generic:Conn_01x06
- SW1, SW10, SW11, SW12, SW13, SW14, SW15, SW16, SW17, SW18, SW19, SW2, SW20, SW21, SW22, SW23, SW24, SW25, SW27, SW28, SW29, SW3, SW4, SW5, SW6, SW7, SW8, SW9: footprint Lily58-footprint:MX_PG1350-Under_FLIP_HOLES_18mm -> Keyboard_Footprints:MX_1U_Flip; symbol Lily58-rescue:SW_PUSH-Lily58-cache -> Keyboard_Symbols:MX_SWITCH
- SW26: symbol Lily58-rescue:SW_PUSH-Lily58-cache -> Keyboard_Symbols:MX_SWITCH
- TH1, TH2: footprint Lily58-footprint:HOLE_M2 -> MountingHole:MountingHole_2.2mm_M2_Pad; symbol Lily58-rescue:HOLE-Lily58-cache -> Mechanical:MountingHole
- TH3, TH4, TH5, TH6, TH7: footprint Lily58-footprint:HOLE_M2_TH -> MountingHole:MountingHole_2.2mm_M2_Pad; symbol Lily58-rescue:HOLE-Lily58-cache -> Mechanical:MountingHole
- gave numbers to parts that had none: 1
Connections:
- net GND: now also U2.15 (GND), U2.23 (GND), U2.35 (GND), U2.43 (GND), U2.5 (UGND), J0.5 (GND), J0.6 (Shield), U0.2 (GND)
- net RESET: now also U2.13 (~RESET)
- net SCL: now also U2.18 (PD0)
- net SDA: now also U2.19 (PD1)
- net VCC: now also U2.14 (VCC), U2.2 (UVCC), U2.24 (AVCC), U2.34 (VCC), U2.44 (AVCC), F0.1, R0.1, U0.5 (VBUS)
- net col0: now also U2.37 (PF6)
- net col1: now also U2.36 (PF7)
- net col2: now also U2.9 (PB1)
- net col3: now also U2.11 (PB3)
- net col4: now also U2.10 (PB2)
- net col5: now also U2.30 (PB6)
- net row0: now also U2.31 (PC6)
- net row1: now also U2.27 (PD7)
- net row2: now also U2.1 (PE6)
- net row3: now also U2.28 (PB4)
- net row4: now also U2.29 (PB5)
- new net USB_D+: J0.3 (D+), R0.2, U0.1 (I/O1), U0.6 (I/O1)
- new net USB_D-: J0.2 (D-), U0.3 (I/O2), U0.4 (I/O2)
- new net VBUS: F0.2, J0.1 (VBUS)
- no-connect marks 4 -> 5
Other:
- moved on the sheet: D1, D10, D11, D12, D13, D14, D15, D16, D17, D18, D19, D2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

Commit message: Updated layout to use more comps
Need to do ATMEGA32U4 circuitry still
Parts:
- removed JP1, JP2, JP3, JP4, JP5, JP6, JP7, JP8: Jumper_NO_Small, Lily58-footprint:Jumper, symbol Device:Jumper_NO_Small
- removed P4: OLED, Lily58-footprint:MY_SIL-4, symbol Lily58-rescue:CONN_01X04-Lily58-cache
- added SHT1, SHT2, SHT3, SHT4, SHT5, SHT6, SHT7, SHT8: R, Keyboard_Footprints:C_0603, symbol Device:R
- added SW30: Rotary_Encoder_Switch, Keyboard_Footprints:EC11E, symbol Device:Rotary_Encoder_Switch
- DISP0: footprint Keyboard_Footprints:OLED -> Keyboard_Footprints:OLED_128x32
- RSW1: footprint Lily58-footprint:TACT_SWITCH_TVBP06 -> Keyboard_Footprints:SPST_FSM2JRT
- SW26: footprint Lily58-footprint:MX_PG1350-Under_FLIP_HOLES_27mm -> Keyboard_Footprints:MX_1.5U_Flip
Connections:
- net GND: now also SHT2.2, SHT7.2, SW30.C
- net SCL: now also SHT3.2, SHT6.2
- net SDA: now also SHT1.2, SHT8.2
- net USB_D+: now also U2.4 (D+)
- net USB_D-: now also U2.3 (D-)
- net VCC: now also SHT4.2, SHT5.2
- net col5: now also SW30.S1
- net at D25.2, SW25.2: now also SW30.S2
- net at DISP0.1 (GND): now also SHT7.1, SHT8.1
- net at DISP0.2 (VCC): now also SHT5.1, SHT6.1
- net at DISP0.3 (SCL): now also SHT3.1, SHT4.1
- net at DISP0.4 (SDA): now also SHT1.1, SHT2.1
- new net ROTA: SW30.A
- new net ROTB: SW30.B
Other:
- note added: "Right Side, use 0 ohm resistors for SHT1, SHT3, SHT5, SHT7\n\nLeft Side, use 0 ohm resistors for SHT2, SHT4, SHT6, SHT8"
- moved on the sheet: D25, D26, D27, D28, D29, J2, P1, P2, U1, W1

Commit message: Updated ATMEGA32U4 schematic
Parts:
- removed P3: ICSP, Lily58-footprint:ICSP, symbol Connector_Generic:Conn_01x06
- removed U1: ProMicro, Lily58-footprint:ProMicro_rev2, symbol Lily58-rescue:ProMicro_2-Lily58-cache
- added C? (x2): 22pF, symbol Device:C_Small
- added C?: 1uF, symbol Device:C_Small
- added C? (x4): 0.1uF, symbol Device:C_Small
- added C?: 10uF, symbol Device:C_Small
- added J?: ICSP, Connector_PinHeader_2.54mm:PinHeader_2x03_P2.54mm_Vertical, symbol Connector_Generic:Conn_02x03_Odd_Even
- added J?: AudioJack4, symbol Connector:AudioJack4
- added JP?: Jumper_NC_Dual, Jumper:SolderJumper-3_P1.3mm_Open_Pad1.0x1.5mm, symbol Device:Jumper_NC_Dual
- added R?: 10k, Keyboard_Footprints:R_0603, symbol Device:R_Small_US
- added Y?: XTAL, symbol Device:Crystal_GND24_Small
- SW30: value Rotary_Encoder_Switch -> EC11E
Connections:
- net labels added: Data, OLED_SCL, OLED_SDA, SIDE_DETECT, XTAL1, XTAL2
- net labels removed: LED, RST
- wire segments 287 -> 316
- no-connect marks 5 -> 2
Other:
- note added: "Left Side"
- note added: "Right Side"
- moved on the sheet: J2, P1, P2, RSW1, SW30, U2, W1
