File: pcb/Lily58.sch (KiCad schematic (older format))
At the start: 84 parts, among them J1 LED, J2 4PIN, P1 i2c_pin, P2 i2c_pin, P3 ICSP, P4 OLED, SW1 SW_PUSH, SW10 SW_PUSH, SW11 SW_PUSH, SW12 SW_PUSH, SW13 SW_PUSH, SW14 SW_PUSH, SW15 SW_PUSH, SW16 SW_PUSH, SW17 SW_PUSH, SW18 SW_PUSH, SW19 SW_PUSH, SW2 SW_PUSH, SW20 SW_PUSH, SW21 SW_PUSH, SW22 SW_PUSH, SW23 SW_PUSH, SW24 SW_PUSH, SW25 SW_PUSH, SW26 SW_PUSH, SW27 SW_PUSH, SW28 SW_PUSH, SW29 SW_PUSH, SW3 SW_PUSH, SW4 SW_PUSH, SW5 SW_PUSH, SW6 SW_PUSH, SW7 SW_PUSH, SW8 SW_PUSH, SW9 SW_PUSH, U1 ProMicro

Commit message: Start of update to use my library and re-route
Parts:
- removed J1: LED, Lily58-footprint:StripLED, symbol Lily58-cache:LED
- removed JP1, JP2, JP3, JP4, JP5, JP6, JP7, JP8: Jumper_NO_Small, Lily58-footprint:Jumper, symbol Device:Jumper_NO_Small
- removed P1, P2: i2c_pin, Lily58-footprint:1pin_conn, symbol Lily58-cache:i2c_pin
- removed P4: OLED, Lily58-footprint:MY_SIL-4, symbol Lily58-cache:CONN_01X04
- added W2: I2C_jmp_CLK, Lily58-footprint:jumper_data, symbol Device:Jumper
- added W3: I2C_jmp_SDA, Lily58-footprint:jumper_data, symbol Device:Jumper
- D1, D10, D11, D12, D13, D14, D15, D16, D17, D18, D19, D2, D20, D21, D22, D23, D24, D25, D26, D27, D28, D29, D3, D4, D5, D6, D7, D8, D9: footprint Lily58-footprint:Diode_TH_SOD123 -> Keyboard_Footprints:D_SOD-123; symbol Lily58-cache:D -> Device:D_Small
- J2: symbol Lily58-cache:MJ-4PP-9 -> Lily58-rescue:MJ-4PP-9-Lily58-cache
- P3: symbol Lily58-cache:CONN_01X06 -> Lily58-rescue:CONN_01X06-Lily58-cache
- R1, R2: value R -> 4.7k; footprint Lily58-footprint:RESISTOR_mini -> Keyboard_Footprints:R_0603; symbol Lily58-cache:R -> Device:R_Small_US
- RSW1: symbol Lily58-cache:SW_RST -> Lily58-rescue:SW_RST-Lily58-cache
- SW1, SW10, SW11, SW12, SW13, SW14, SW15, SW16, SW17, SW18, SW19, SW2, SW20, SW21, SW22, SW23, SW24, SW25, SW27, SW28, SW29, SW3, SW4, SW5, SW6, SW7, SW8, SW9: footprint Lily58-footprint:MX_PG1350-Under_FLIP_HOLES_18mm -> Keyboard_Footprints:MX_1U; symbol Lily58-cache:SW_PUSH -> Switch:SW_Push
- SW26: symbol Lily58-cache:SW_PUSH -> Switch:SW_Push
- TH1, TH2, TH3, TH4, TH5, TH6, TH7: symbol Lily58-cache:HOLE -> Mechanical:MountingHole
- U1: footprint Lily58-footprint:ProMicro_rev2 -> Keyboard_Footprints:ProMicro_rev; symbol Lily58-cache:ProMicro_2 -> Lily58-rescue:ProMicro_2-Lily58-cache
- W1: value jumper -> RX_jmp
Connections:
- wire segments 84 -> 202
Other:
- note added: "Arduino Pro Micro / Elite-C Interface\n"
- note added: "Controller Circuitry"
- moved on the sheet: W1

Commit message: Update comps
Parts:
- added J?: AudioJack4, symbol Connector:AudioJack4
- added JP?: R1_BOT, symbol Device:Jumper_NC_Small
- added JP?: R1_TOP, symbol Device:Jumper_NC_Small
- added JP?: R2_TOP, symbol Device:Jumper_NC_Small
- added JP?: R2_BOT, symbol Device:Jumper_NC_Small
- added R?: 4.7k, Keyboard_Footprints:R_0603, symbol Device:R_Small_US
Connections:
- net GND: now also J?.S
- net SCL: now also JP?.1, JP?.2; no longer R2.2
- net SDA: now also JP?.1, JP?.2
- net VCC: now also J?.T, R?.1
- net sp_data: now reaches J2.3, W1.2, W3.2
- net sp_clk: now reaches J2.4, W2.2
- net LED: no longer names the net of U1.1 (TX(PD3))
- new net: J?.R2, JP?.1, JP?.1, R2.2
- new net: J?.R1, JP?.2, JP?.2, R?.2
- no-connect marks 4 -> 5
Other:
- moved on the sheet: J2, R1, R2, W1, W2, W3
